Commit message: prepare to add C++ version

File: urdf/cassie_Lpinned_original.urdf (robot description, URDF)
Before this commit: robot cassie, 17 links, 16 joints
Joints:
- joint hip_abduction_right: origin xyz=0 0 -0.07 rpy=0 -1.5707963267948966192313216916398 0 -> xyz=0 0 -0.07 rpy=0 -1.57079632679 0
- joint hip_rotation_right: origin xyz=0 0 -0.09 rpy=0 1.5707963267948966192313216916398 -1.5707963267948966192313216916398 -> xyz=0 0 -0.09 rpy=0 1.57079632679 -1.57079632679

File: urdf/rabbit_pinned - Copy.urdf (robot description, URDF)
Before this commit: robot rabbit_pinned, 5 links, 4 joints
Joints:
- joint q1_left: origin xyz=0 0 0 rpy=0 0 0.1 -> xyz=0 0 0 rpy=0 0 0
- joint q1_right: origin xyz=0 0 0.4 rpy=0 0 0.3 -> xyz=0 0 0.4 rpy=0 0 0
- joint q2_left: origin xyz=0 0 0.4 rpy=0 0.2 0 -> xyz=0 0 0.4 rpy=0 0 0
- joint q2_right: origin xyz=0 0 0.4 rpy=0.1 0.2 0 -> xyz=0 0 0.4 rpy=0 0 0
